File: watch.kicad_pcb (KiCad board)
At the start: 2 copper layers, 60.6 x 53.2 mm, 80 parts, among them M1 3V3 35mA, Q1 IRLML6302, Q2 IRLML0060TRPbF, SW1 B3U-3000P, SW2 B3U-3000P, SW3 B3U-3000P, SW4 B3U-3000P, SW5 B3U-3000P, X1 MICROSD_SPI, X2 209E-BE01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

Commit message: PCB Changed
Parts:
- BT1: footprint Resistors_SMD:R_0805_HandSoldering -> Capacitors_SMD:C_1206; moved to B.Cu
- C1, C3: footprint Capacitors_SMD:C_0805 -> Capacitors_SMD:C_1206; moved to B.Cu
- C2, C20, C22, C6, C8, D1, DD2, R17, R2: moved to B.Cu
- moved X2 267.7 mm to (293.5, 80.5), turned to 90 degrees
- moved R14 196.8 mm to (291.5, 80.2), turned to 180 degrees
- moved DD2 190.2 mm to (248.2, 76.5), turned to 180 degrees
- moved R10 173.1 mm to (291.5, 81.5), turned to 180 degrees
- moved X3 166.9 mm to (191.0, 53.5), turned to 90 degrees
- moved R11 163.1 mm to (280.5, 76.8), turned to 180 degrees
- moved X1 151.9 mm to (238.0, 141.0)
- moved R12 148.2 mm to (280.5, 79.5)
- moved R5 145.9 mm to (267.5, 113.2)
- moved C21 141.4 mm to (250.2, 77.0), turned to 270 degrees
- moved C23 132.1 mm to (248.2, 75.0)
- moved R17 130.4 mm to (247.8, 80.0), turned to 135 degrees
- moved DD4 113.1 mm to (248.2, 77.0), turned to 90 degrees
- moved DA3 68.8 mm to (158.0, 70.5), turned to 180 degrees
- moved C22 68.7 mm to (187.0, 125.8)
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Routing:
- net GND: track 40.7 -> 89.0 mm, vias 17 -> 21
- net VCC: track 5.94 -> 34.2 mm
- net +5V: track 0.00 -> 11.1 mm, vias 0 -> 2
- net VEE: track 0.00 -> 9.97 mm, vias 0 -> 1
- net /I2C_SCL: track 0.00 -> 7.14 mm, vias 0 -> 2
- net /I2C_SDA: track 0.00 -> 6.12 mm
- net +BATT: track 0.00 -> 5.18 mm, vias 0 -> 1
- net Net-(DA1-Pad5): track 0.00 -> 3.93 mm
- net /~STDBY: track 0.00 -> 3.43 mm
- net /BMC_INT3: track 0.00 -> 3.16 mm
- net /USB_DM: track 0.00 -> 3.10 mm
- net Net-(DD1-Pad44): track 0.00 -> 2.92 mm, vias 0 -> 1
- net /~CHRG: track 0.00 -> 2.83 mm
- net /BMC_INT2: track 0.00 -> 2.64 mm
- net /BMC_INT1: track 0.00 -> 2.64 mm
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Other:
- board size 60.6 x 53.2 mm -> 59.6 x 41.2 mm

Commit message: PCB finished, some changes in schematic
Parts:
- removed C11, C18: 100n, Capacitors_SMD:C_0402
- removed C7: 10n, Capacitors_SMD:C_0402
- removed C9: 10u, Capacitors_SMD:C_0805
- removed L1: fcm1608-0603, Resistors_SMD:R_0603
- removed R1, R29, R3, R30, R4, R5, R6, R7, R8: 10K, Resistors_SMD:R_0402
- removed R9: 470K, Resistors_SMD:R_0402
- removed SW4, SW5: B3U-3000P, Footprints:B3U-3000P
- removed X1: MICROSD_SPI, Footprints:112J-TDAR-R01
- added REF**: Hole, Footprints:Hole, F.Cu at (32.0, 32.0)
- added REF**: Hole, Footprints:Hole, F.Cu at (55.5, 32.0)
- added REF**: Hole, Footprints:Hole, F.Cu at (32.0, 56.0)
- added REF**: Hole, Footprints:Hole, F.Cu at (55.5, 56.0)
- C12, C14, C15, C16, C17, C19, L2, R17, R25: moved to F.Cu
- M1, R11, R12, R21, R22, R23, R26, R27, R28, SP1: moved to B.Cu
- R24: footprint Resistors_SMD:R_0402 -> Resistors_SMD:R_0603
- moved X2 243.1 mm to (53.2, 43.8)
- moved R10 242.9 mm to (51.4, 44.6)
- moved R14 242.9 mm to (51.4, 43.6)
- moved R12 230.0 mm to (53.2, 44.6), turned to 90 degrees
- moved R11 229.8 mm to (53.2, 42.8), turned to 90 degrees
- moved DA4 218.5 mm to (43.8, 49.5)
- moved C15 210.6 mm to (40.0, 40.8), turned to 180 degrees
- moved C12 210.1 mm to (38.8, 49.0), turned to 180 degrees
- moved R17 208.7 mm to (42.9, 40.2), turned to 270 degrees
- moved C21 208.4 mm to (45.5, 38.2)
- moved DD2 208.2 mm to (43.8, 37.2)
- moved DD4 208.1 mm to (43.8, 38.2)
- moved C23 208.1 mm to (43.8, 36.5)
- moved DD1 208.0 mm to (43.8, 45.2)
- moved C17 206.7 mm to (46.2, 49.5), turned to 180 degrees
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Connections:
- DA1 pad 4: /~WALL -> Net-(DA1-Pad4)
- DA4 pad A2: VAA -> /REF
- DA4 pad B2: VAA -> /REF
- DD1 pad 10: /TEMP -> /BTN0
- DD1 pad 11: Net-(DD1-Pad11) -> /BTN1
- DD1 pad 12: /BTN1 -> /BTN2
- DD1 pad 13: /~SC_CD -> Net-(DD1-Pad13)
- DD1 pad 14: /~SD_SS -> Net-(DD1-Pad14)
- DD1 pad 15: /SD_SCK -> Net-(DD1-Pad15)
- DD1 pad 16: /SD_MISO -> /POWER
- DD1 pad 17: /SD_MOSI -> Net-(DD1-Pad17)
- DD1 pad 18: /BTN2 -> /REF
- DD1 pad 19: /BTN3 -> /TEMP
- DD1 pad 2: /BTN0 -> Net-(DD1-Pad2)
- DD1 pad 20: /BTN4 -> Net-(DD1-Pad20)
- DD1 pad 21: /BEEP -> Net-(DD1-Pad21)
- DD1 pad 22: /VIBRO -> Net-(DD1-Pad22)
- DD1 pad 25: /POWER -> /VIBRO
- DD1 pad 26: /~WALL -> Net-(DD1-Pad26)
- DD1 pad 27: /~CHRG -> /~STDBY
- DD1 pad 28: /~STDBY -> /~CHRG
- DD1 pad 38: Net-(DD1-Pad38) -> /BEEP
Routing:
- net GND: track 89.0 -> 259.0 mm, vias 21 -> 33
- net VCC: track 34.2 -> 144.3 mm, vias 3 -> 8
- net /BT_RX: track 1.45 -> 22.0 mm, vias 0 -> 1
- net /I2C_SDA: track 6.12 -> 26.3 mm, vias 0 -> 3
- net Net-(C18-Pad2): track 0.00 -> 19.4 mm, vias 0 -> 1
- net /~RES: track 2.64 -> 21.6 mm, vias 0 -> 2
- net /BT_TX: track 1.45 -> 20.4 mm, vias 0 -> 1
- net +5V: track 11.1 -> 29.5 mm
- net /BTN0: track 3.64 -> 21.8 mm, vias 0 -> 3
- net /BEEP: track 0.00 -> 16.5 mm, vias 0 -> 3
- net /BTN1: track 0.00 -> 14.1 mm, vias 0 -> 1
- net /I2C_SCL: track 7.14 -> 20.9 mm, vias 2 -> 4
- net /BTN2: track 0.00 -> 13.0 mm, vias 0 -> 1
- net /~CHRG: track 2.83 -> 14.9 mm, vias 0 -> 2
- net /VIBRO: track 0.00 -> 10.8 mm, vias 0 -> 1
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- added copper zone on B.Cu, net GND
- added copper zone on F.Cu, net GND
Other:
- board size 59.6 x 41.2 mm -> 27.5 x 28.5 mm
- board text removed: "Copyright (c) 2016 Sviatoslav Semchyshyn"
